File: steno.kicad_sch (KiCad schematic)
At the start: 49 parts, among them SW1 MX_Switch, SW10 MX_Switch, SW11 MX_Switch, SW12 MX_Switch, SW13 MX_Switch, SW14 MX_Switch, SW15 MX_Switch, SW16 MX_Switch, SW17 MX_Switch, SW18 MX_Switch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

Commit message: Update PCB schematics to ECSKv2 design
Connections:
- net C1: now also U1.10 (GPIO7); no longer U1.31 (GPIO26_ADC0)
- net C10: now also U1.17 (GPIO13); no longer U1.24 (GPIO18)
- net C2: now also U1.12 (GPIO9); no longer U1.29 (GPIO22)
- net C3: now also U1.22 (GPIO17); no longer U1.19 (GPIO14)
- net C4: now also U1.24 (GPIO18); no longer U1.17 (GPIO13)
- net C5: now also U1.25 (GPIO19); no longer U1.16 (GPIO12)
- net C6: now also U1.26 (GPIO20); no longer U1.15 (GPIO11)
- net C7: now also U1.14 (GPIO10); no longer U1.27 (GPIO21)
- net C8: now also U1.15 (GPIO11); no longer U1.26 (GPIO20)
- net C9: now also U1.16 (GPIO12); no longer U1.25 (GPIO19)
- net R1: now also U1.7 (GPIO5); no longer U1.34 (GPIO28_ADC2)
- net R2: now also U1.9 (GPIO6); no longer U1.32 (GPIO27_ADC1)
- net R3: now also U1.21 (GPIO16); no longer U1.20 (GPIO15)
Changed lines of the file:
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@@
     )
   )
-  (symbol (lib_id "MCU_RaspberryPi_and_Boards:Pico") (at 64.77 149.86 0) (unit 1)
+  (symbol (lib_id "MCU_RaspberryPi_and_Boards:Pico") (at 64.77 149.86 0) (mirror y) (unit 1)
     (in_bom yes) (on_board yes) (dnp no)
-    (property "Reference" "U1" (at 62.865 119.38 0)
+    (property "Reference" "U1" (at 66.675 119.38 0)
       (effects (font (size 1.27 1.27)) (justify left))
     )
-    (property "Value" "Pico" (at 62.23 121.92 0)
+    (property "Value" "Pico" (at 67.31 121.92 0)
       (effects (font (size 1.27 1.27)) (justify left))
     )
